Commit message: city map added, fixed navigation issue

File: description/robot_core.xacro (robot description, xacro)
@@ -49,5 +49,5 @@
         <parent link="base_link"/>
         <child link="chassis"/>
-        <origin xyz="${-chassis_length/2} 0 0"/>
+        <origin xyz="${-chassis_length/2} 0 ${-wheel_radius/2}"/>
     </joint>
     <link name="chassis">
